File: Design/LLD_Design/V1.0/Project_OAK_MAIN_BRD_V1.0/OAK_Led-Matrix.sch (KiCad schematic (older format))
At the start: 48 parts

Commit message: layout update in progress
Parts:
- gave numbers to parts that had none: 48

Commit message: OAK V1.0 main board routing complete
Other:
- moved on the sheet: C14, C15, C16, C17, C18, C19, D10, D11, D12, D13, D14, D15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
